File: hardware/CANberry/CANberry.kicad_sch (KiCad schematic)
At the start: 42 parts, among them J1 USB_C_Receptacle_USB2.0, J2 0393570003, J3 M20-9990346, J4 SWD, SW1 KMR2, U1 AP2112K-3.3, U2 USBLC6-2SC6, U3 ADM3053, U4 STM32F072C8Tx

Commit message: rename to CANberry due to name colision
Parts:
- added LOGO1: Logo_Open_Hardware_Small, josh-logos:OSHW_Logo_3.6x3.6_F.Mask, symbol Graphic:Logo_Open_Hardware_Small
- C1: value 1u -> 4u7; LCSC C1592 -> (none); MPN  CL10A105KO8NNNC -> (none); Manufacturer Samsung Electro-Mechanicsr -> (none)
- C11, C4: LCSC (none) -> C84416; MPN (none) -> GRM21BR61E106KA73L; Manufacturer (none) -> Murata Electronics
- C12, C13, C14, C15: LCSC C14663 -> (none); MPN CL10B104KB8NNNCr -> (none); Manufacturer Samsung Electro-Mechanicsr -> (none)
- C2, C3: value 1u -> 4u7; LCSC C15849 -> (none); MPN CL10A105MP8NNNC r -> (none); Manufacturer Samsung Electro-Mechanicsr -> (none)
- C8: value 1u -> 4u7
- D1: value LED -> RED
- D2: value LED -> GRN
- D3: LCSC (none) -> C970030; MPN (none) -> ESDCAN24-2BLY; Manufacturer (none) -> STMicroelectronics
- H1, H2, H3, H4: DNP (none) -> DNP; now left out of the parts list
- J1: MPN (none) -> TYPE-C-31-M-14; MPN  TYPE-C-31-M-14 -> (none)
- J2: value 0393570003 -> 1751251; LCSC (none) -> C91152; MPN (none) -> 1751251; Manufacturer (none) -> Phoenix Contact
- J4: now left out of the parts list
- R1, R2: LCSC C14677 -> (none); MPN  RC0603JR-075K1L -> (none); Manufacturer YAGEO -> (none)
- SW1: LCSC (none) -> C72443; MPN (none) -> KMR221GLFS; Manufacturer (none) -> C&K
- U2: MPN (none) -> USBLC6-2SC6; MPN  USBLC6-2SC6 -> (none)
- U3: LCSC (none) -> C117821; MPN (none) -> ADM3053
Other:
- note added: "2-3 Terminates CAN bus"
- note removed: "1-2 Terminates CAN bus"
- title: CANcat -> CANberry
